File: sparrow_v1_pcb/esp-break.sch (KiCad schematic (older format))
At the start: 29 parts, among them J1 Conn_02x03_Odd_Even, J2 Conn_02x05_Odd_Even, J3 Conn_01x06, J4 Conn_01x01, J5 Conn_01x06, J7 Conn_01x02_Male, J8 USB_B_Micro, SW1 SW_Push, U1 ESP32-WROOM-32, U2 AP1117-33

Commit message: Updated the lables for First and Second version of the Board (Coin and Washing) and Readme. Next Step: Logo and Labels placement
Parts:
- C1, C4: value C -> 22uf
- C2, C3, C5, C6: value C -> 0.1uf
- R1: value R -> 10k
- R2: value R -> 330
- RF12: renamed from R12; value R -> 0
- RF5: renamed from R5; value R -> 0
- RF7: renamed from R7; value R -> 0
- RF9: renamed from R9; value R -> 0
- RS10: renamed from R10; value R -> 0
- RS11: renamed from R11; value R -> 0
- RS3: renamed from R3; value 200k -> 220k
- RS4: renamed from R4; value 85k -> 120k
- RS6: renamed from R6; value R -> 0
- RS8: renamed from R8; value R -> 0
Changed lines of the file:
@@
 P 6250 4000
 F 0 "C2" H 6428 4046 50  0000 L CNN
-F 1 "C" H 6428 3955 50  0000 L CNN
+F 1 "0.1uf" H 6428 3955 50  0000 L CNN
 F 2 "Capacitor_SMD:C_1206_3216Metric" H 6250 4000 50  0001 C CNN
 F 3 "~" H 6250 4000 50  0001 C CNN
@@
 P 5800 4000
 F 0 "C1" H 5978 4046 50  0000 L CNN
-F 1 "C" H 5978 3955 50  0000 L CNN
+F 1 "22uf" H 5978 3955 50  0000 L CNN
 F 2 "Capacitor_SMD:C_1206_3216Metric" H 5800 4000 50  0001 C CNN
 F 3 "~" H 5800 4000 50  0001 C CNN
@@
 P 7550 4000
 F 0 "C4" H 7728 4046 50  0000 L CNN
-F 1 "C" H 7728 3955 50  0000 L CNN
+F 1 "22uf" H 7728 3955 50  0000 L CNN
 F 2 "Capacitor_SMD:C_1206_3216Metric" H 7550 4000 50  0001 C CNN
 F 3 "~" H 7550 4000 50  0001 C CNN
@@
 P 7100 4000
 F 0 "C3" H 7278 4046 50  0000 L CNN
-F 1 "C" H 7278 3955 50  0000 L CNN
+F 1 "0.1uf" H 7278 3955 50  0000 L CNN
 F 2 "Capacitor_SMD:C_1206_3216Metric" H 7100 4000 50  0001 C CNN
 F 3 "~" H 7100 4000 50  0001 C CNN
@@
 P 4300 4350
 F 0 "R1" H 4370 4396 50  0000 L CNN
-F 1 "R" H 4370 4305 50  0000 L CNN
+F 1 "10k" H 4370 4305 50  0000 L CNN
 F 2 "Resistor_SMD:R_1206_3216Metric" V 4230 4350 50  0001 C CNN
 F 3 "~" H 4300 4350 50  0001 C CNN
@@
 3.3
 $Comp
-L Device:R R6
+L Device:R RS6
 U 1 1 5DD02A1E
 P 6200 2600
-F 0 "R6" H 6270 2646 50  0000 L CNN
-F 1 "R" H 6270 2555 50  0000 L CNN
+F 0 "RS6" H 6270 2646 50  0000 L CNN
+F 1 "0" H 6270 2555 50  0000 L CNN
 F 2 "Resistor_SMD:R_1206_3216Metric" V 6130 2600 50  0001 C CNN
 F 3 "~" H 6200 2600 50  0001 C CNN
@@
 $EndComp
 $Comp
-L Device:R R9
+L Device:R RF9
 U 1 1 5DD09723
 P 6500 2300
-F 0 "R9" H 6570 2346 50  0000 L CNN
-F 1 "R" H 6570 2255 50  0000 L CNN
+F 0 "RF9" H 6570 2346 50  0000 L CNN
+F 1 "0" H 6570 2255 50  0000 L CNN
 F 2 "Resistor_SMD:R_1206_3216Metric" V 6430 2300 50  0001 C CNN
 F 3 "~" H 6500 2300 50  0001 C CNN
@@
 $EndComp
 $Comp
-L Device:R R11
+L Device:R RS11
 U 1 1 5DD09CF1
 P 6800 2600
-F 0 "R11" H 6870 2646 50  0000 L CNN
-F 1 "R" H 6870 2555 50  0000 L CNN
+F 0 "RS11" H 6870 2646 50  0000 L CNN
+F 1 "0" H 6870 2555 50  0000 L CNN
 F 2 "Resistor_SMD:R_1206_3216Metric" V 6730 2600 50  0001 C CNN
 F 3 "~" H 6800 2600 50  0001 C CNN
@@
 io19
 $Comp
-L Device:R R8
+L Device:R RS8
 U 1 1 5DD0EBB8
 P 6500 2100
-F 0 "R8" H 6570 2146 50  0000 L CNN
-F 1 "R" H 6570 2055 50  0000 L CNN
+F 0 "RS8" H 6570 2146 50  0000 L CNN
+F 1 "0" H 6570 2055 50  0000 L CNN
 F 2 "Resistor_SMD:R_1206_3216Metric" V 6430 2100 50  0001 C CNN
 F 3 "~" H 6500 2100 50  0001 C CNN
@@
 $EndComp
 $Comp
-L Device:R R5
+L Device:R RF5
 U 1 1 5DD0EF8A
 P 5850 2100
-F 0 "R5" H 5920 2146 50  0000 L CNN
-F 1 "R" H 5920 2055 50  0000 L CNN
+F 0 "RF5" H 5920 2146 50  0000 L CNN
+F 1 "0" H 5920 2055 50  0000 L CNN
 F 2 "Resistor_SMD:R_1206_3216Metric" V 5780 2100 50  0001 C CNN
 F 3 "~" H 5850 2100 50  0001 C CNN
@@
 $EndComp
 $Comp
-L Device:R R12
+L Device:R RF12
 U 1 1 5DD102EF
 P 7150 2100
-F 0 "R12" H 7220 2146 50  0000 L CNN
-F 1 "R" H 7220 2055 50  0000 L CNN
+F 0 "RF12" H 7220 2146 50  0000 L CNN
+F 1 "0" H 7220 2055 50  0000 L CNN
 F 2 "Resistor_SMD:R_1206_3216Metric" V 7080 2100 50  0001 C CNN
 F 3 "~" H 7150 2100 50  0001 C CNN
@@
 	6300 1900 6450 1900
 $Comp
-L Device:R R7
+L Device:R RF7
 U 1 1 5DD12A1D
 P 6450 1550
-F 0 "R7" H 6520 1596 50  0000 L CNN
-F 1 "R" H 6520 1505 50  0000 L CNN
+F 0 "RF7" H 6520 1596 50  0000 L CNN
+F 1 "0" H 6520 1505 50  0000 L CNN
 F 2 "Resistor_SMD:R_1206_3216Metric" V 6380 1550 50  0001 C CNN
 F 3 "~" H 6450 1550 50  0001 C CNN
@@
 $EndComp
 $Comp
-L Device:R R10
+L Device:R RS10
 U 1 1 5DD13336
 P 6550 1550
-F 0 "R10" H 6400 1600 50  0000 L CNN
-F 1 "R" H 6450 1500 50  0000 L CNN
+F 0 "RS10" H 6400 1600 50  0000 L CNN
+F 1 "0" H 6450 1500 50  0000 L CNN
 F 2 "Resistor_SMD:R_1206_3216Metric" V 6480 1550 50  0001 C CNN
 F 3 "~" H 6550 1550 50  0001 C CNN
@@
 	6500 1400 6550 1400
 $Comp
-L Device:R R3
+L Device:R RS3
 U 1 1 5DD196F3
 P 5750 2400
-F 0 "R3" H 5820 2446 50  0000 L CNN
-F 1 "200k" H 5820 2355 50  0000 L CNN
+F 0 "RS3" H 5820 2446 50  0000 L CNN
+F 1 "220k" H 5820 2355 50  0000 L CNN
 F 2 "Resistor_SMD:R_1206_3216Metric" V 5680 2400 50  0001 C CNN
 F 3 "~" H 5750 2400 50  0001 C CNN
@@
 $EndComp
 $Comp
-L Device:R R4
+L Device:R RS4
 U 1 1 5DD19EFE
 P 5750 2800
-F 0 "R4" H 5820 2846 50  0000 L CNN
-F 1 "85k" H 5820 2755 50  0000 L CNN
+F 0 "RS4" H 5820 2846 50  0000 L CNN
+F 1 "120k" H 5820 2755 50  0000 L CNN
 F 2 "Resistor_SMD:R_1206_3216Metric" V 5680 2800 50  0001 C CNN
 F 3 "~" H 5750 2800 50  0001 C CNN
@@
 P 4300 3950
 F 0 "C5" H 4478 3996 50  0000 L CNN
-F 1 "C" H 4478 3905 50  0000 L CNN
+F 1 "0.1uf" H 4478 3905 50  0000 L CNN
 F 2 "Capacitor_SMD:C_1206_3216Metric" H 4300 3950 50  0001 C CNN
 F 3 "~" H 4300 3950 50  0001 C CNN
@@
 P 4300 2650
 F 0 "R2" H 4370 2696 50  0000 L CNN
-F 1 "R" H 4370 2605 50  0000 L CNN
+F 1 "330" H 4370 2605 50  0000 L CNN
 F 2 "Resistor_SMD:R_1206_3216Metric" V 4230 2650 50  0001 C CNN
 F 3 "~" H 4300 2650 50  0001 C CNN
@@
 P 4800 4450
 F 0 "C6" H 4978 4496 50  0000 L CNN
-F 1 "C" H 4978 4405 50  0000 L CNN
+F 1 "0.1uf" H 4978 4405 50  0000 L CNN
 F 2 "Capacitor_SMD:C_1206_3216Metric" H 4800 4450 50  0001 C CNN
 F 3 "~" H 4800 4450 50  0001 C CNN

Commit message: Changed the location of the vias from the footprint of the tagconnect and updated the version patch number
Connections:
- net labels added: RX2, TX2
- wire segments 56 -> 60
Changed lines of the file:
@@
 EESchema Schematic File Version 4
-LIBS:esp-break-cache
 EELAYER 30 0
 EELAYER END
@@
 Text GLabel 4150 2650 0    50   Input ~ 0
 led
-Text GLabel 3300 2850 2    50   Input ~ 0
+Text GLabel 3600 3150 2    50   Input ~ 0
 led
 Wire Wire Line
@@
 Text GLabel 3300 3150 2    50   Input ~ 0
 io21
-Text GLabel 3300 3250 2    50   Input ~ 0
+Text GLabel 3600 3250 2    50   Input ~ 0
 io22
 Text GLabel 3300 3450 2    50   Input ~ 0
@@
 	6700 2200 6300 2200
 Text GLabel 7300 2100 2    50   Input ~ 0
-tx
+TX2
 Text GLabel 5700 2100 0    50   Input ~ 0
-rx
+RX2
 $Comp
 L Regulator_Linear:AP1117-33 U2
@@
 Text GLabel 8350 4200 0    50   Input ~ 0
 adc3
+Wire Wire Line
+	3600 3250 3550 3250
+Wire Wire Line
+	3600 3150 3550 3150
+Wire Wire Line
+	3550 3150 3550 3250
+Connection ~ 3550 3250
+Wire Wire Line
+	3550 3250 3300 3250
+Text GLabel 3300 2850 2    50   Input ~ 0
+RX2
+Text GLabel 3300 2750 2    50   Input ~ 0
+TX2
 $EndSCHEMATC
