File: sparrow_v1_pcb/esp-break.sch (KiCad schematic (older format))
At the start: 28 parts, among them J1 Conn_02x03_Odd_Even, Q1 BSS138, Q2 BSS138, SW1 SW_Push, U1 ESP32-WROOM-32D, U2 LD1117S33TR_SOT223, U3 TPS62153

Commit message: Updated Library and removed internal power and updated footprints
Parts:
- removed C7: 10 uF, Capacitor_SMD:C_1210_3225Metric, symbol Device:C
- removed C8: 3.3 nF, Capacitor_SMD:C_0603_1608Metric, symbol Device:C
- removed C9: 22 uF, Capacitor_SMD:C_0805_2012Metric, symbol Device:C
- removed L1: 2.2 uH, Inductor_SMD:L_Coilcraft_XxL4020, symbol Device:L
- removed R7: 100k, Resistor_SMD:R_0201_0603Metric, symbol Device:R
- removed U3: TPS62153, Package_DFN_QFN:VQFN-16-1EP_3x3mm_P0.5mm_EP1.68x1.68mm_ThermalVias, symbol Regulator_Switching:TPS62153
- C1, C2, C3, C4, C5, C6: footprint Capacitor_SMD:C_0201_0603Metric -> Capacitor_SMD:C_0805_2012Metric_Pad1.18x1.45mm_HandSolder
- D1: footprint LED_SMD:LED_0201_0603Metric -> LED_SMD:LED_0805_2012Metric_Pad1.15x1.40mm_HandSolder
- PWR2: symbol Connector:USB_B_Micro -> esp-break-rescue:USB_B_Micro-Connector
- R1, R2, R3, R4, R5, R6: footprint Resistor_SMD:R_0201_0603Metric -> Resistor_SMD:R_0805_2012Metric_Pad1.20x1.40mm_HandSolder
Connections:
- net Vout is gone; now on net vcc: C1.1, C2.1, U2.3 (VI)
- net vcc: no longer IN1.1 (Pin_1), OUT1.1 (Pin_1)
- new net: IN1.1 (Pin_1), OUT1.1 (Pin_1)
Changed lines of the file:
@@
 EESchema Schematic File Version 4
-LIBS:esp-break-cache
 EELAYER 30 0
 EELAYER END
@@
 F 0 "C2" H 6578 3146 50  0000 L CNN
 F 1 "0.1uf" H 6578 3055 50  0000 L CNN
-F 2 "Capacitor_SMD:C_0201_0603Metric" H 6400 3100 50  0001 C CNN
+F 2 "Capacitor_SMD:C_0805_2012Metric_Pad1.18x1.45mm_HandSolder" H 6400 3100 50  0001 C CNN
 F 3 "~" H 6400 3100 50  0001 C CNN
 	1    6400 3100
@@
 F 0 "C1" H 6128 3146 50  0000 L CNN
 F 1 "22uf" H 6128 3055 50  0000 L CNN
-F 2 "Capacitor_SMD:C_0201_0603Metric" H 5950 3100 50  0001 C CNN
+F 2 "Capacitor_SMD:C_0805_2012Metric_Pad1.18x1.45mm_HandSolder" H 5950 3100 50  0001 C CNN
 F 3 "~" H 5950 3100 50  0001 C CNN
 	1    5950 3100
@@
 F 0 "C4" H 7878 3146 50  0000 L CNN
 F 1 "22uf" H 7878 3055 50  0000 L CNN
-F 2 "Capacitor_SMD:C_0201_0603Metric" H 7700 3100 50  0001 C CNN
+F 2 "Capacitor_SMD:C_0805_2012Metric_Pad1.18x1.45mm_HandSolder" H 7700 3100 50  0001 C CNN
 F 3 "~" H 7700 3100 50  0001 C CNN
 	1    7700 3100
@@
 Connection ~ 6850 3500
 $Comp
-L Connector:USB_B_Micro PWR2
+L esp-break-rescue:USB_B_Micro-Connector PWR2
 U 1 1 5DBA3F97
 P 2250 4250
@@
 Text GLabel 2250 4650 3    50   Input ~ 0
 gnd
-Text GLabel 6400 2800 1    50   Input ~ 0
-Vout
 Text GLabel 2600 800  2    50   Input ~ 0
 3.3
@@
 F 0 "C3" H 7428 3146 50  0000 L CNN
 F 1 "0.1uf" H 7428 3055 50  0000 L CNN
-F 2 "Capacitor_SMD:C_0201_0603Metric" H 7250 3100 50  0001 C CNN
+F 2 "Capacitor_SMD:C_0805_2012Metric_Pad1.18x1.45mm_HandSolder" H 7250 3100 50  0001 C CNN
 F 3 "~" H 7250 3100 50  0001 C CNN
 	1    7250 3100
@@
 F 0 "R1" H 4370 4396 50  0000 L CNN
 F 1 "10k" H 4370 4305 50  0000 L CNN
-F 2 "Resistor_SMD:R_0201_0603Metric" V 4230 4350 50  0001 C CNN
+F 2 "Resistor_SMD:R_0805_2012Metric_Pad1.20x1.40mm_HandSolder" V 4230 4350 50  0001 C CNN
 F 3 "~" H 4300 4350 50  0001 C CNN
 	1    4300 4350
@@
 F 0 "D1" H 4593 2395 50  0000 C CNN
 F 1 "LED" H 4593 2486 50  0000 C CNN
-F 2 "LED_SMD:LED_0201_0603Metric" H 4600 2650 50  0001 C CNN
+F 2 "LED_SMD:LED_0805_2012Metric_Pad1.15x1.40mm_HandSolder" H 4600 2650 50  0001 C CNN
 F 3 "~" H 4600 2650 50  0001 C CNN
 	1    4600 2650
@@
 F 0 "C5" H 4478 3996 50  0000 L CNN
 F 1 "0.1uf" H 4478 3905 50  0000 L CNN
-F 2 "Capacitor_SMD:C_0201_0603Metric" H 4300 3950 50  0001 C CNN
+F 2 "Capacitor_SMD:C_0805_2012Metric_Pad1.18x1.45mm_HandSolder" H 4300 3950 50  0001 C CNN
 F 3 "~" H 4300 3950 50  0001 C CNN
 	1    4300 3950
@@
 F 0 "R2" H 4370 2696 50  0000 L CNN
 F 1 "330" H 4370 2605 50  0000 L CNN
-F 2 "Resistor_SMD:R_0201_0603Metric" V 4230 2650 50  0001 C CNN
+F 2 "Resistor_SMD:R_0805_2012Metric_Pad1.20x1.40mm_HandSolder" V 4230 2650 50  0001 C CNN
 F 3 "~" H 4300 2650 50  0001 C CNN
 	1    4300 2650
@@
 F 0 "C6" H 4978 4496 50  0000 L CNN
 F 1 "0.1uf" H 4978 4405 50  0000 L CNN
-F 2 "Capacitor_SMD:C_0201_0603Metric" H 4800 4450 50  0001 C CNN
+F 2 "Capacitor_SMD:C_0805_2012Metric_Pad1.18x1.45mm_HandSolder" H 4800 4450 50  0001 C CNN
 F 3 "~" H 4800 4450 50  0001 C CNN
 	1    4800 4450
@@
 F 0 "R3" H 5770 1046 50  0000 L CNN
 F 1 "10k" H 5770 955 50  0000 L CNN
-F 2 "Resistor_SMD:R_0201_0603Metric" V 5630 1000 50  0001 C CNN
+F 2 "Resistor_SMD:R_0805_2012Metric_Pad1.20x1.40mm_HandSolder" V 5630 1000 50  0001 C CNN
 F 3 "~" H 5700 1000 50  0001 C CNN
 	1    5700 1000
@@
 F 0 "R4" H 6270 1046 50  0000 L CNN
 F 1 "10k" H 6270 955 50  0000 L CNN
-F 2 "Resistor_SMD:R_0201_0603Metric" V 6130 1000 50  0001 C CNN
+F 2 "Resistor_SMD:R_0805_2012Metric_Pad1.20x1.40mm_HandSolder" V 6130 1000 50  0001 C CNN
 F 3 "~" H 6200 1000 50  0001 C CNN
 	1    6200 1000
@@
 F 0 "R5" H 7420 1046 50  0000 L CNN
 F 1 "10k" H 7420 955 50  0000 L CNN
-F 2 "Resistor_SMD:R_0201_0603Metric" V 7280 1000 50  0001 C CNN
+F 2 "Resistor_SMD:R_0805_2012Metric_Pad1.20x1.40mm_HandSolder" V 7280 1000 50  0001 C CNN
 F 3 "~" H 7350 1000 50  0001 C CNN
 	1    7350 1000
@@
 F 0 "R6" H 7920 1046 50  0000 L CNN
 F 1 "10k" H 7920 955 50  0000 L CNN
-F 2 "Resistor_SMD:R_0201_0603Metric" V 7780 1000 50  0001 C CNN
+F 2 "Resistor_SMD:R_0805_2012Metric_Pad1.20x1.40mm_HandSolder" V 7780 1000 50  0001 C CNN
 F 3 "~" H 7850 1000 50  0001 C CNN
 	1    7850 1000
@@
 NoConn ~ 2000 2700
 $Comp
-L Regulator_Switching:TPS62153 U3
-U 1 1 5F00BF3A
-P 6900 4700
-F 0 "U3" H 6900 5381 50  0000 C CNN
-F 1 "TPS62153" H 6900 5290 50  0000 C CNN
-F 2 "Package_DFN_QFN:VQFN-16-1EP_3x3mm_P0.5mm_EP1.68x1.68mm_ThermalVias" H 7050 4250 50  0001 L CNN
-F 3 "http://www.ti.com/lit/ds/symlink/TPS62150.pdf" H 6900 4700 50  0001 C CNN
-	1    6900 4700
-	1    0    0    -1
-$EndComp
-Text GLabel 7000 3900 1    50   Input ~ 0
-vcc
-Wire Wire Line
-	6500 4500 6500 4200
-Wire Wire Line
-	6500 4200 6800 4200
-Wire Wire Line
-	6800 4200 7000 4200
-Connection ~ 6800 4200
-Wire Wire Line
-	7000 4200 7000 4000
-Connection ~ 7000 4200
-$Comp
-L Device:C C8
-U 1 1 5F0139AE
-P 6350 4600
-F 0 "C8" V 6098 4600 50  0000 C CNN
-F 1 "3.3 nF" V 6189 4600 50  0000 C CNN
-F 2 "Capacitor_SMD:C_0603_1608Metric" H 6388 4450 50  0001 C CNN
-F 3 "~" H 6350 4600 50  0001 C CNN
-	1    6350 4600
-	0    1    1    0
-$EndComp
-Wire Wire Line
-	6200 4600 6100 4600
-Text GLabel 6100 4700 3    50   Input ~ 0
-gnd
-Wire Wire Line
-	6100 4700 6100 4600
-Connection ~ 6100 4600
-Wire Wire Line
-	6100 4600 5950 4600
-$Comp
-L Device:C C7
-U 1 1 5F0181AC
-P 6100 4350
-F 0 "C7" H 6215 4396 50  0000 L CNN
-F 1 "10 uF" H 6215 4305 50  0000 L CNN
-F 2 "Capacitor_SMD:C_1210_3225Metric" H 6138 4200 50  0001 C CNN
-F 3 "~" H 6100 4350 50  0001 C CNN
-	1    6100 4350
-	1    0    0    -1
-$EndComp
-Wire Wire Line
-	6100 4500 6100 4600
-Wire Wire Line
-	6100 4200 6100 4000
-Wire Wire Line
-	6100 4000 7000 4000
-Connection ~ 7000 4000
-Wire Wire Line
-	7000 4000 7000 3900
-Wire Wire Line
-	6500 4700 6500 4750
-Wire Wire Line
-	6500 4750 6400 4750
-Wire Wire Line
-	6400 4750 6400 4800
-Connection ~ 6500 4750
-Wire Wire Line
-	6500 4750 6500 4800
-Text GLabel 6400 4800 3    50   Input ~ 0
-gnd
-Wire Wire Line
-	6800 5200 6800 5400
-Wire Wire Line
-	6800 5400 7000 5400
-Wire Wire Line
-	7000 5400 7000 5200
-Wire Wire Line
-	7300 4900 7300 5400
-Wire Wire Line
-	7300 5400 7000 5400
-Connection ~ 7000 5400
-Text GLabel 7000 5400 3    50   Input ~ 0
-gnd
-Wire Wire Line
-	7300 4700 7800 4700
-Wire Wire Line
-	7800 4700 7800 4500
-$Comp
-L Device:R R7
-U 1 1 5F02689D
-P 7900 4650
-F 0 "R7" H 7970 4696 50  0000 L CNN
-F 1 "100k" H 7970 4605 50  0000 L CNN
-F 2 "Resistor_SMD:R_0201_0603Metric" V 7830 4650 50  0001 C CNN
-F 3 "~" H 7900 4650 50  0001 C CNN
-	1    7900 4650
-	1    0    0    -1
-$EndComp
-Wire Wire Line
-	7300 4800 7900 4800
-Wire Wire Line
-	7800 4500 7900 4500
-Wire Wire Line
-	7900 4500 8200 4500
-Connection ~ 7900 4500
-$Comp
-L Device:C C9
-U 1 1 5F02D11A
-P 8200 4700
-F 0 "C9" H 8315 4746 50  0000 L CNN
-F 1 "22 uF" H 8315 4655 50  0000 L CNN
-F 2 "Capacitor_SMD:C_0805_2012Metric" H 8238 4550 50  0001 C CNN
-F 3 "~" H 8200 4700 50  0001 C CNN
-	1    8200 4700
-	1    0    0    -1
-$EndComp
-Wire Wire Line
-	8200 4500 8200 4550
-Text GLabel 8200 4900 3    50   Input ~ 0
-gnd
-Wire Wire Line
-	8200 4850 8200 4900
-$Comp
-L Device:L L1
-U 1 1 5F032225
-P 7550 4500
-F 0 "L1" V 7740 4500 50  0000 C CNN
-F 1 "2.2 uH" V 7649 4500 50  0000 C CNN
-F 2 "Inductor_SMD:L_Coilcraft_XxL4020" H 7550 4500 50  0001 C CNN
-F 3 "~" H 7550 4500 50  0001 C CNN
-	1    7550 4500
-	0    -1   -1   0
-$EndComp
-Wire Wire Line
-	7300 4500 7400 4500
-Wire Wire Line
-	7700 4500 7800 4500
-Connection ~ 7800 4500
-Text GLabel 8250 4500 2    50   Output ~ 0
-Vout
-Wire Wire Line
-	8200 4500 8250 4500
-Connection ~ 8200 4500
-Text GLabel 6900 5200 3    50   Output ~ 0
-gnd
-Text GLabel 10100 3150 2    50   Input ~ 0
-vcc
-Wire Wire Line
-	9750 3150 10100 3150
-Connection ~ 9750 3150
-$Comp
 L Regulator_Linear:LD1117S33TR_SOT223 U2
 U 1 1 5F0B3AAC
@@
 	1    0    0    -1
 $EndComp
+Text GLabel 6400 2750 1    50   Input ~ 0
+vcc
+Wire Wire Line
+	6400 2800 6400 2750
 $EndSCHEMATC
