File: sparrow_v1_pcb/_autosave-esp-break.sch (KiCad schematic (older format))
At the start: 28 parts, among them J1 Conn_02x03_Odd_Even, Q1 BSS138, Q2 BSS138, SW1 SW_Push, U1 ESP32-WROOM-32D, U2 LD1117S33TR_SOT223, U3 TPS62153

Commit message: Updated the PCB layout with vias and LDO footprint
Parts:
- C8: footprint Capacitor_SMD:C_0402_1005Metric -> Capacitor_SMD:C_0603_1608Metric
Changed lines of the file:
@@
 F 0 "C8" V 6098 4600 50  0000 C CNN
 F 1 "3.3 nF" V 6189 4600 50  0000 C CNN
-F 2 "Capacitor_SMD:C_0402_1005Metric" H 6388 4450 50  0001 C CNN
+F 2 "Capacitor_SMD:C_0603_1608Metric" H 6388 4450 50  0001 C CNN
 F 3 "~" H 6350 4600 50  0001 C CNN
 	1    6350 4600
