File: sparrow_pcb_proj/esp-break.sch (KiCad schematic (older format))
At the start: 22 parts, among them J1 Conn_02x03_Odd_Even, Q1 BSS138, Q2 BSS138, SW1 SW_Push, U1 ESP32-WROOM-32D, U2 LD1117S33TR_SOT223

Commit message: After PCB Check by Ovee
Parts:
- U1: symbol RF_Module:ESP32-WROOM-32D -> esp-break-rescue:ESP32-WROOM-32D-RF_Module
Changed lines of the file:
@@
 EESchema Schematic File Version 4
+LIBS:esp-break-cache
 EELAYER 30 0
 EELAYER END
@@
 $EndDescr
 $Comp
-L RF_Module:ESP32-WROOM-32D U1
+L esp-break-rescue:ESP32-WROOM-32D-RF_Module U1
 U 1 1 5DB6DAA1
 P 2600 2200
